File: 2023_ROBOCON_B_CHIKU.sch (EAGLE design)
At the start: 22 parts, among them CON1 XT90PW-F, CON2 XT90PW-M, U1 TLP-250

Commit message: Chiku version
Parts:
- removed CON1: XT90PW-F, amass:XT90PW-F
- removed CON2: XT90PW-M, amass:XT90PW-M
- removed IRLB-3: IRLB3813STAND, OKUDA_libraries:IRLB3813STAND
- added C3: 330F, capacitor-wima:C2,5-3
- added C4: 10uF, capacitor-wima:C2,5-3
- added C5: 1uF, capacitor-wima:C2,5-3
- added C8: (no value), capacitor-wima:C2,5-3
- added CTRL, EMERGENCY1, SERVO_CONECT: 02-JST, con-jst-xh_1:02-JST
- added FAN, FAN1, FAN2: (no value), con-jst-xh_1:03-JST
- added JP1, JP2, JP3: (no value), pinhead:PINHD-1X2
- added LED, LED2: (no value), con-jst-xh_1:04-JST
- added LED3, LED6: (no value), led:LED5MM
- added LED4, LED5, LED7: (no value), led:LED3MM
- added LIPO-BATTERY: XT90PB-F, amass:XT90PB-F
- added R3, R6: 1k, resistor:R-EU_0207/12
- added R5, R7, R8: 1K, resistor:R-EU_0204/5
- added U$2: F446RE, F446RE_ver1.4:F446RE
- added U$5: TWELITE-PIN, TWELITE_ver1.2 (1):TWELITE-PIN
- added U$6: HINATA, HINATA:HINATA
- C1: value 1uF -> (none)
- C2: value 0.1uF -> 330F
- R2: value 10k -> 10K; device resistor:R-EU_0207/7 -> resistor:R-EU_0204/5
Connections:
- removed net MD_GND: CON1.-, IRLB-3.D
- new net 3V3: C1.1, U$2.3V3, U$5.VCC
- new net 5V(U5V): U$2.USV, U$6.+5V
- new net CS: U$2.PB_9, U$6.CS
- new net GND1: C1.2, U$2.GND6, U$5.GND1
- new net GND2: U$2.GND2, U$6.GND5
- new net GND3: SERVO_CONECT.1, U$2.GND3
- new net GND4: LED4.C, LED5.C, LED7.C, U$2.GND
- new net LED: U$2.PC_8, U$6.LED
- new net LED1: R5.2, U$2.PA_5
- new net LED2: R7.2, U$2.PA_6
- new net LED3: R8.2, U$2.PA_7
- new net MC_RX: U$2.PC_10, U$5.TX
- new net MC_TX: U$2.PC_11, U$5.RX
- new net MISO: U$2.PB_15, U$6.MISO
- new net MOSI: U$2.PC_1, U$6.MOSI
- new net N$1: LED6.A, R6.1
- new net N$11: LED5.A, R7.1
- new net N$14: LED7.A, R8.1
- new net N$3: LED3.A, R3.1
- new net N$6: LED4.A, R5.1
- new net PWM: SERVO_CONECT.2, U$2.PB_7
- new net SCK: U$2.PC_7, U$6.SCK
- net +12V: now also FAN.2, FAN1.2, FAN2.2, LED.4, LED2.4
- net BLUE: now also LED.1, LED2.1
- net GND: now also C3.1, C4.1, C5.1, C8.2, JP2.2, LIPO-BATTERY.-; no longer C1.1, CON2.-, IRLB-3.S
- net GREEN: now also LED.3, LED2.3
- net LED_GND: now also FAN.3, FAN1.3, FAN2.3, LED6.C
- net N$10: now also CTRL.2, EMERGENCY1.1
- net N$2: now also CTRL.1, JP2.1
- net N$7: no longer IRLB-3.G
- net RED: now also LED.2, LED2.2
- net SERVO_GND: now also LED3.C
- net VCC: now also C3.2, C4.2, C5.2, C8.1, EMERGENCY1.2, LIPO-BATTERY.+, R3.2, R6.2; no longer C1.2, CON1.+, CON2.+
Other:
- note added: "FAN LED"
- note added: "Nch MOSFET"
- note added: "hinata"
- note removed: "LED"
- note removed: "to MD10c"
